File: wifi-page.kicad_pcb (KiCad board)
At the start: 4 copper layers, 64.5 x 28 mm, 44 parts, among them J1 USB_B_Micro, J2 Conn_01x04, SW1 SW_Push, SW2 SW_Push, U1 ESP32-S3-WROOM-1, U2 AP2112K-3.3, U3 CAT24C256

Commit message: update silkscreen
Parts:
- moved FID1 1.82 mm to (197.2, 61.4)
- moved G*** 1.20 mm to (193.6, 60.1)
Other:
- board text added: "BOOT"
- board text added: "EN"
- board text added: "GND"
- board text added: "RX"
- board text added: "TX"
Changed lines of the file:
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@@
 		(tags "tactile switch kmr2")
 		(property "Reference" "SW1"
-			(at -1.527 -2.6 0)
+			(at 2 -2.6 0)
 			(layer "F.SilkS")
 			(effects
@@
 	(footprint "Fiducial:Fiducial_1mm_Mask2mm"
 		(layer "F.Cu")
-		(at 199 61.1)
+		(at 197.2 61.35)
 		(descr "Fiducial, circular marking, 1mm bare copper, 2mm soldermask opening (Level A)")
 		(tags "fiducial")
 		(property "Reference" "FID1"
-			(at 0 -1.95 0)
+			(at 0.65 -2.05 0)
 			(layer "F.SilkS")
 			(effects
@@
 	(footprint "LOGO"
 		(layer "F.Cu")
-		(at 194.31 59.182)
+		(at 193.6 60.15)
 		(property "Reference" "G***"
 			(at 0 0 0)
@@
 		(tags "tactile switch kmr2")
 		(property "Reference" "SW2"
-			(at -1 -2.6 0)
+			(at 4.25 -2.3 0)
 			(layer "F.SilkS")
 			(effects
@@
 		(layer "Edge.Cuts")
 	)
+	(gr_text "GND"
+		(at 198.6 65.05 0)
+		(layer "F.SilkS")
+		(effects
+			(font
+				(size 1 1)
+				(thickness 0.2)
+				(bold yes)
+			)
+			(justify left bottom)
+		)
+	)
+	(gr_text "TX"
+		(at 199.85 57.05 0)
+		(layer "F.SilkS")
+		(effects
+			(font
+				(size 1 1)
+				(thickness 0.2)
+				(bold yes)
+			)
+			(justify left bottom)
+		)
+	)
+	(gr_text "RX"
+		(at 199.8 61 0)
+		(layer "F.SilkS")
+		(effects
+			(font
+				(size 1 1)
+				(thickness 0.2)
+				(bold yes)
+			)
+			(justify left bottom)
+		)
+	)
+	(gr_text "BOOT"
+		(at 200.85 53.15 0)
+		(layer "F.SilkS")
+		(effects
+			(font
+				(size 1 1)
+				(thickness 0.2)
+				(bold yes)
+			)
+			(justify left bottom)
+		)
+	)
+	(gr_text "EN"
+		(at 202.65 47.75 0)
+		(layer "F.SilkS")
+		(effects
+			(font
+				(size 1 1)
+				(thickness 0.2)
+				(bold yes)
+			)
+			(justify left bottom)
+		)
+	)
 	(gr_text "3v3 SDA SCL GND"
